Commit message: big changes

File: GEN3-7DOF-NOVISION_FOR_URDF_ARM_V12.urdf (robot description, URDF)
Before this commit: robot GEN3-7DOF-NOVISION_FOR_URDF_ARM_V12, 9 links, 8 joints
Links:
- link base_link: geometry collision mesh filename=base_link.STL; visual mesh filename=base_link.STL
- link bracelet_link: geometry collision mesh filename=bracelet_no_vision_link.STL; visual mesh filename=bracelet_no_vision_link.STL
- link forearm_link: geometry collision mesh filename=forearm_link.STL; visual mesh filename=forearm_link.STL
- link half_arm_1_link: geometry collision mesh filename=half_arm_1_link.STL; visual mesh filename=half_arm_1_link.STL
- link half_arm_2_link: geometry collision mesh filename=half_arm_2_link.STL; visual mesh filename=half_arm_2_link.STL
- link shoulder_link: geometry collision mesh filename=shoulder_link.STL; visual mesh filename=shoulder_link.STL
- link spherical_wrist_1_link: geometry collision mesh filename=spherical_wrist_1_link.STL; visual mesh filename=spherical_wrist_1_link.STL
- link spherical_wrist_2_link: geometry collision mesh filename=spherical_wrist_2_link.STL; visual mesh filename=spherical_wrist_2_link.STL

File: gen3_2f85.urdf (robot description, URDF)
Before this commit: robot gen3_, 31 links, 30 joints
Links:
- removed link wrist_camera_link
- removed link wrist_camera_mount_link
- removed link wrist_mounted_camera_bottom_screw_frame
- removed link wrist_mounted_camera_color_frame
- removed link wrist_mounted_camera_color_optical_frame
- removed link wrist_mounted_camera_depth_frame
- removed link wrist_mounted_camera_depth_optical_frame
- removed link wrist_mounted_camera_infra1_frame
- removed link wrist_mounted_camera_infra1_optical_frame
- removed link wrist_mounted_camera_infra2_frame
- removed link wrist_mounted_camera_infra2_optical_frame
- removed link wrist_mounted_camera_link
- link gen3_base_link: geometry collision mesh filename=base_link.stl; visual mesh filename=base_link.stl
- link gen3_bracelet_link: geometry collision mesh filename=bracelet_no_vision_link.stl; visual mesh filename=bracelet_no_vision_link.stl
- link gen3_forearm_link: geometry collision mesh filename=forearm_link.stl; visual mesh filename=forearm_link.stl
- link gen3_half_arm_1_link: geometry collision mesh filename=half_arm_1_link.stl; visual mesh filename=half_arm_1_link.stl
- link gen3_half_arm_2_link: geometry collision mesh filename=half_arm_2_link.stl; visual mesh filename=half_arm_2_link.stl
- link gen3_robotiq_85_base_link: geometry collision mesh filename=robotiq_base.stl; visual mesh filename=robotiq_base.stl
- link gen3_robotiq_85_left_finger_link: geometry collision mesh filename=left_finger.stl; visual mesh filename=left_finger.stl
- link gen3_robotiq_85_left_finger_tip_link: geometry collision mesh filename=left_finger_tip.stl; visual mesh filename=left_finger_tip.stl
- link gen3_robotiq_85_left_inner_knuckle_link: geometry collision mesh filename=left_inner_knuckle.stl; visual mesh filename=left_inner_knuckle.stl
- link gen3_robotiq_85_left_knuckle_link: geometry collision mesh filename=left_knuckle.stl; visual mesh filename=left_knuckle.stl
- link gen3_robotiq_85_right_finger_link: geometry collision mesh filename=right_finger.stl; visual mesh filename=right_finger.stl
- link gen3_robotiq_85_right_finger_tip_link: geometry collision mesh filename=right_finger_tip.stl; visual mesh filename=right_finger_tip.stl
- link gen3_robotiq_85_right_inner_knuckle_link: geometry collision mesh filename=right_inner_knuckle.stl; visual mesh filename=right_inner_knuckle.stl
- link gen3_robotiq_85_right_knuckle_link: geometry collision mesh filename=right_knuckle.stl; visual mesh filename=right_knuckle.stl
- link gen3_shoulder_link: geometry collision mesh filename=shoulder_link.stl; visual mesh filename=shoulder_link.stl
- link gen3_spherical_wrist_1_link: geometry collision mesh filename=spherical_wrist_1_link.stl; visual mesh filename=spherical_wrist_1_link.stl
- link gen3_spherical_wrist_2_link: geometry collision mesh filename=spherical_wrist_2_link.stl; visual mesh filename=spherical_wrist_2_link.stl
Joints:
- removed joint wrist_camera_joint
- removed joint wrist_camera_mount_joint
- removed joint wrist_mounted_camera_color_joint
- removed joint wrist_mounted_camera_color_optical_joint
- removed joint wrist_mounted_camera_depth_joint
- removed joint wrist_mounted_camera_depth_optical_joint
- removed joint wrist_mounted_camera_infra1_joint
- removed joint wrist_mounted_camera_infra1_optical_joint
- removed joint wrist_mounted_camera_infra2_joint
- removed joint wrist_mounted_camera_infra2_optical_joint
- removed joint wrist_mounted_camera_joint
- removed joint wrist_mounted_camera_link_joint
