Commit message: big changes

File: gen3_2f85.urdf (robot description, URDF)
Before this commit: robot gen3_, 19 links, 18 joints
Links:
- added link table, mass 200; collision box size=2.4 1.6 0.06; visual box size=2.4 1.6 0.06
Joints:
- added joint world_to_table: type fixed, parent world, child table, origin xyz=0 0 0 rpy=0 0 0
- joint gen3_base_joint: parent world -> table

Commit message: new

File: gen3_2f85.urdf (robot description, URDF)
Before this commit: robot gen3_, 20 links, 19 joints
Links:
- added link wrist_camera_link
- added link wrist_camera_mount_link, mass 0.5; collision mesh filename=bracelet_with_vision_link.stl; visual mesh filename=bracelet_with_vision_link.stl
- added link wrist_mounted_camera_bottom_screw_frame
- added link wrist_mounted_camera_color_frame
- added link wrist_mounted_camera_color_optical_frame
- added link wrist_mounted_camera_depth_frame
- added link wrist_mounted_camera_depth_optical_frame
- added link wrist_mounted_camera_infra1_frame
- added link wrist_mounted_camera_infra1_optical_frame
- added link wrist_mounted_camera_infra2_frame
- added link wrist_mounted_camera_infra2_optical_frame
- added link wrist_mounted_camera_link, mass 0.072; collision box size=0.02005 0.099 0.023; visual mesh filename=d415.stl
Joints:
- added joint wrist_camera_joint: type fixed, parent gen3_bracelet_link, child wrist_camera_link, origin xyz=0 -0.06841 -0.05044 rpy=0 1.7444444444444447 -1.5708
- added joint wrist_camera_mount_joint: type fixed, parent gen3_bracelet_link, child wrist_camera_mount_link, origin xyz=0 0 0.0 rpy=0 0 0
- added joint wrist_mounted_camera_color_joint: type fixed, parent wrist_mounted_camera_link, child wrist_mounted_camera_color_frame, origin xyz=0 0.015 0 rpy=0 0 0
- added joint wrist_mounted_camera_color_optical_joint: type fixed, parent wrist_mounted_camera_color_frame, child wrist_mounted_camera_color_optical_frame, origin xyz=0 0 0 rpy=-1.5707963267948966 0 -1.5707963267948966
- added joint wrist_mounted_camera_depth_joint: type fixed, parent wrist_mounted_camera_link, child wrist_mounted_camera_depth_frame, origin xyz=0 0 0 rpy=0 0 0
- added joint wrist_mounted_camera_depth_optical_joint: type fixed, parent wrist_mounted_camera_depth_frame, child wrist_mounted_camera_depth_optical_frame, origin xyz=0 0 0 rpy=-1.5707963267948966 0 -1.5707963267948966
- added joint wrist_mounted_camera_infra1_joint: type fixed, parent wrist_mounted_camera_link, child wrist_mounted_camera_infra1_frame, origin xyz=0 0.0 0 rpy=0 0 0
- added joint wrist_mounted_camera_infra1_optical_joint: type fixed, parent wrist_mounted_camera_infra1_frame, child wrist_mounted_camera_infra1_optical_frame, origin xyz=0 0 0 rpy=-1.5707963267948966 0 -1.5707963267948966
- added joint wrist_mounted_camera_infra2_joint: type fixed, parent wrist_mounted_camera_link, child wrist_mounted_camera_infra2_frame, origin xyz=0 -0.055 0 rpy=0 0 0
- added joint wrist_mounted_camera_infra2_optical_joint: type fixed, parent wrist_mounted_camera_infra2_frame, child wrist_mounted_camera_infra2_optical_frame, origin xyz=0 0 0 rpy=-1.5707963267948966 0 -1.5707963267948966
- added joint wrist_mounted_camera_joint: type fixed, parent wrist_camera_link, child wrist_mounted_camera_bottom_screw_frame, origin xyz=0 0 0 rpy=0 0 0
- added joint wrist_mounted_camera_link_joint: type fixed, parent wrist_mounted_camera_bottom_screw_frame, child wrist_mounted_camera_link, origin xyz=0 0.02 0.0115 rpy=0 0 0
